File: Updated 75 key.kicad_pcb (KiCad board)
At the start: 2 copper layers, 298 x 108 mm, 151 parts, among them K1 KEYSW, K10 KEYSW, K11 KEYSW, K12 KEYSW, K13 KEYSW, K14 KEYSW, K15 KEYSW, K16 KEYSW, K17 KEYSW, K18 KEYSW, K19 KEYSW, K2 KEYSW, K20 KEYSW, K21 KEYSW, K22 KEYSW, K23 KEYSW, K24 KEYSW, K25 KEYSW, K26 KEYSW, K27 KEYSW, K28 KEYSW, K29 KEYSW, K3 KEYSW, K30 KEYSW, K31 KEYSW, K32 KEYSW, K33 KEYSW, K34 KEYSW, K35 KEYSW, K36 KEYSW, K37 KEYSW, K38 KEYSW, K39 KEYSW, K4 KEYSW, K40 KEYSW, K41 KEYSW, K42 KEYSW, K43 KEYSW, K44 KEYSW, K45 KEYSW, K46 KEYSW, K47 KEYSW, K48 KEYSW, K49 KEYSW, K5 KEYSW, K50 KEYSW, K51 KEYSW, K52 KEYSW, K53 KEYSW, K54 KEYSW, K55 KEYSW, K56 KEYSW, K57 KEYSW, K58 KEYSW, K59 KEYSW, K6 KEYSW, K60 KEYSW, K61 KEYSW, K62 KEYSW, K63 KEYSW, K64 KEYSW, K65 KEYSW, K66 KEYSW, K67 KEYSW, K68 KEYSW, K69 KEYSW, K7 KEYSW, K70 KEYSW, K71 KEYSW, K72 KEYSW, K73 KEYSW, K74 KEYSW, K75 KEYSW, K8 KEYSW, K9 KEYSW, U1 ProMicro

Commit message: Add files via upload
Parts:
- added REF**: MountingHole_6.5mm, MountingHole:MountingHole_6.5mm, F.Cu at (57.9, 128.0)
- added REF**: MountingHole_6.5mm, MountingHole:MountingHole_6.5mm, F.Cu at (154.9, 128.0)
- added REF**: MountingHole_6.5mm, MountingHole:MountingHole_6.5mm, F.Cu at (249.9, 128.0)
- added REF**: MountingHole_6.5mm, MountingHole:MountingHole_6.5mm, F.Cu at (346.9, 128.0)
- added REF**: MountingHole_6.5mm, MountingHole:MountingHole_6.5mm, F.Cu at (346.9, 227.0)
- added REF**: MountingHole_6.5mm, MountingHole:MountingHole_6.5mm, F.Cu at (249.9, 227.0)
- added REF**: MountingHole_6.5mm, MountingHole:MountingHole_6.5mm, F.Cu at (154.9, 227.0)
- added REF**: MountingHole_6.5mm, MountingHole:MountingHole_6.5mm, F.Cu at (57.9, 227.0)
- moved D1 105.8 mm to (68.0, 144.0)
- moved D10 105.8 mm to (240.8, 144.1)
- moved D11 105.8 mm to (260.0, 144.1)
- moved D12 105.8 mm to (279.4, 144.1)
- moved D13 105.8 mm to (298.6, 144.1)
- moved D14 105.8 mm to (317.9, 144.1)
- moved D15 105.8 mm to (337.1, 144.1)
- moved D16 105.8 mm to (68.1, 163.2)
- moved D17 105.8 mm to (87.3, 163.2)
- moved D18 105.8 mm to (106.5, 163.2)
- moved D19 105.8 mm to (125.6, 163.2)
- moved D2 105.8 mm to (87.2, 144.0)
- moved D20 105.8 mm to (144.9, 163.2)
- moved D21 105.8 mm to (164.2, 163.2)
- moved D22 105.8 mm to (183.3, 163.2)
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Routing:
- net Net-(K12-Pad1): track 59.9 -> 583.0 mm, vias 0 -> 8
- net Net-(K11-Pad1): track 82.1 -> 541.7 mm, vias 0 -> 4
- net Net-(K14-Pad1): track 26.3 -> 476.2 mm, vias 0 -> 4
- net Net-(K17-Pad1): track 90.9 -> 527.2 mm, vias 1 -> 7
- net Net-(K13-Pad1): track 25.5 -> 456.3 mm, vias 1 -> 6
- net Net-(K15-Pad1): track 66.3 -> 484.0 mm, vias 0 -> 8
- net Net-(K1-Pad1): track 86.0 -> 502.4 mm, vias 1 -> 5
- net Net-(K16-Pad1): track 72.5 -> 452.7 mm, vias 0 -> 6
- net Net-(K18-Pad1): track 120.0 -> 487.1 mm, vias 2 -> 4
- net Net-(D28-Pad1): track 145.5 -> 364.1 mm, vias 0 -> 4
- net Net-(D10-Pad1): track 122.8 -> 327.1 mm, vias 0 -> 2
- net Net-(D37-Pad1): track 166.3 -> 298.7 mm
- net Net-(D46-Pad1): track 165.0 -> 261.1 mm
- net Net-(D19-Pad1): track 166.1 -> 222.7 mm, vias 0 -> 2
- net Net-(D1-Pad1): track 195.9 -> 220.2 mm, vias 0 -> 1
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- added copper zone on B.Cu, net (none)
- added copper zone on F.Cu, net GND
Other:
- outline, holes or cut-outs redrawn

Commit message: Add files via upload
Routing:
- net GND: track 18.8 -> 18.9 mm, vias 0 -> 3
Changed lines of the file:
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@@
     (thickness 1.6)
     (drawings 8)
-    (tracks 1192)
+    (tracks 1200)
     (zones 0)
     (modules 159)
@@
   (segment (start 90.65625 151.3125) (end 90.65625 152.53125) (width 0.25) (layer B.Cu) (net 93))
   (segment (start 93.1875 155.0625) (end 93.1875 159.233752) (width 0.25) (layer B.Cu) (net 93))
-  (segment (start 94.71375 137.64363) (end 94.71375 136.235) (width 0.25) (layer F.Cu) (net 94))
-  (segment (start 94.71375 138.775) (end 94.71375 137.64363) (width 0.25) (layer F.Cu) (net 94))
-  (segment (start 80.60512 133.695) (end 79.47375 133.695) (width 0.25) (layer F.Cu) (net 94))
-  (segment (start 82.168751 133.695) (end 80.60512 133.695) (width 0.25) (layer F.Cu) (net 94))
-  (segment (start 84.708751 136.235) (end 82.168751 133.695) (width 0.25) (layer F.Cu) (net 94))
-  (segment (start 94.71375 136.235) (end 84.708751 136.235) (width 0.25) (layer F.Cu) (net 94))
+  (via (at 81.5625 133.6875) (size 0.8) (drill 0.4) (layers F.Cu B.Cu) (net 94))
+  (segment (start 79.47375 133.695) (end 81.555 133.695) (width 0.25) (layer F.Cu) (net 94))
+  (segment (start 81.555 133.695) (end 81.5625 133.6875) (width 0.25) (layer F.Cu) (net 94))
+  (via (at 87.28125 134.625) (size 0.8) (drill 0.4) (layers F.Cu B.Cu) (net 94))
+  (segment (start 83.151502 134.625) (end 87.28125 134.625) (width 0.25) (layer B.Cu) (net 94))
+  (segment (start 81.5625 133.6875) (end 82.214002 133.6875) (width 0.25) (layer B.Cu) (net 94))
+  (segment (start 82.214002 133.6875) (end 83.151502 134.625) (width 0.25) (layer B.Cu) (net 94))
+  (segment (start 87.28125 134.625) (end 88.96875 136.3125) (width 0.25) (layer F.Cu) (net 94))
+  (via (at 92.25 136.3125) (size 0.8) (drill 0.4) (layers F.Cu B.Cu) (net 94))
+  (segment (start 88.96875 136.3125) (end 92.25 136.3125) (width 0.25) (layer F.Cu) (net 94))
+  (segment (start 94.63625 136.3125) (end 94.71375 136.235) (width 0.25) (layer B.Cu) (net 94))
+  (segment (start 92.25 136.3125) (end 94.63625 136.3125) (width 0.25) (layer B.Cu) (net 94))
+  (segment (start 94.71375 137.36637) (end 94.71375 138.775) (width 0.25) (layer B.Cu) (net 94))
+  (segment (start 94.71375 136.235) (end 94.71375 137.36637) (width 0.25) (layer B.Cu) (net 94))
   (zone (net 94) (net_name GND) (layer F.Cu) (hatch edge 0.508)
     (connect_pads (clearance 0.508))
